Commit message: actualizacion

File: simple_air_hockey/resources/disco.urdf (robot description, URDF)
Before this commit: robot disco, 4 links, 3 joints
Links:
- link base_link: geometry collision cylinder length=1.0 radius=0.40; visual cylinder length=0.1 radius=0.40

File: simple_air_hockey/resources/mesa.urdf (robot description, URDF)
Before this commit: robot mesa, 26 links, 25 joints
Links:
- link side_wall_1: geometry collision box size=0.56 3.0 17.8; visual box size=0.56 1.5 17.8
- link side_wall_2: geometry collision box size=0.56 3.0 17.8; visual box size=0.56 1.5 17.8
- link side_wall_3_1: geometry collision box size=3.0 1 4.28; visual box size=1.5 1 4.28
- link side_wall_3_2: geometry collision box size=3.0 1 4.28; visual box size=1.5 1 4.28
- link side_wall_3_3: geometry collision box size=0.4 1 2.4; visual box size=0.2 1 2.4
- link side_wall_4_1: geometry collision box size=3.0 1.0 4.28; visual box size=1.5 1.0 4.28
- link side_wall_4_2: geometry collision box size=3.0 1.0 4.28; visual box size=1.5 1.0 4.28
- link side_wall_4_3: geometry collision box size=0.4 1.0 2.4; visual box size=0.2 1.0 2.4

File: simple_air_hockey/resources/scara-left.urdf (robot description, URDF)
Before this commit: robot scara-left, 8 links, 7 joints
Links:
- link arm_1: geometry visual box size=0.4 3.0 0.1
- link arm_2: geometry visual box size=0.4 2.2 0.1
- link base_robot: geometry visual box size=1.5 0.8 0.1
- link end_arm_1: geometry visual cylinder length=0.1 radius=0.35
- link end_arm_2: geometry visual cylinder length=0.4 radius=0.35
- link mallet: geometry collision cylinder length=1.4 radius=0.45; visual cylinder length=0.17 radius=0.45
- link start_arm_1: geometry visual cylinder length=0.1 radius=0.35
- link start_arm_2: geometry visual cylinder length=0.1 radius=0.35

File: simple_air_hockey/resources/scara-right.urdf (robot description, URDF)
Before this commit: robot scara-right, 8 links, 7 joints
Links:
- link arm_1: geometry visual box size=0.4 3.0 0.1
- link arm_2: geometry visual box size=0.4 2.2 0.1
- link base_robot: geometry visual box size=1.5 0.8 0.1
- link end_arm_1: geometry visual cylinder length=0.1 radius=0.35
- link end_arm_2: geometry visual cylinder length=0.4 radius=0.35
- link mallet: geometry collision cylinder length=1.4 radius=0.45; visual cylinder length=0.17 radius=0.45
- link start_arm_1: geometry visual cylinder length=0.1 radius=0.35
- link start_arm_2: geometry visual cylinder length=0.1 radius=0.35
